Commit message: carto

File: description/imu.xacro (robot description, xacro)
@@ -1,35 +1,3 @@
-<?xml version="1.0"?>
-<robot xmlns:xacro="http://www.ros.org/wiki/xacro">
-  <!-- IMU Link -->
-  <link name="imu_link">
-    <visual>
-      <origin xyz="0 0 0" rpy="0 0 0"/>
-      <geometry>
-        <box size="0.03 0.03 0.01"/>
-      </geometry>
-      <material name="black"/>
-    </visual>
-    <collision>
-      <origin xyz="0 0 0" rpy="0 0 0"/>
-      <geometry>
-        <box size="0.03 0.03 0.01"/>
-      </geometry>
-    </collision>
-    <inertial>
-      <mass value="0.01"/>
-      <origin xyz="0 0 0" rpy="0 0 0"/>
-      <inertia
-        ixx="1e-6" ixy="0.0"  ixz="0.0"
-        iyy="1e-6" iyz="0.0"
-        izz="1e-6"/>
-    </inertial>
-  </link>
-  <!-- IMU Joint (fixed to chassis or base_link) -->
-  <joint name="imu_joint" type="fixed">
-    <parent link="chassis"/>
-    <child link="imu_link"/>
-    <origin xyz="0.0 0.0 0.08" rpy="0 0 0"/>
-  </joint>
- <gazebo reference="imu_link">
+<gazebo reference="imu_link">
   <sensor name="imu_sensor" type="imu">
     <always_on>true</always_on>
@@ -38,8 +6,9 @@
     <imu>
       <angular_velocity>
-        <x><noise type="gaussian"><mean>0.0</mean><stddev>0.015</stddev></noise></x>
-        <y><noise type="gaussian"><mean>0.0</mean><stddev>0.015</stddev></noise></y>
-        <z><noise type="gaussian"><mean>0.0</mean><stddev>0.015</stddev></noise></z>
+        <z><noise type="gaussian"><mean>0.0</mean><stddev>0.01</stddev></noise></z>
       </angular_velocity>
+      <orientation>
+        <z><noise type="gaussian"><mean>0.0</mean><stddev>0.001</stddev></noise></z>
+      </orientation>
       <linear_acceleration>
         <x><noise type="gaussian"><mean>0.0</mean><stddev>0.2</stddev></noise></x>
@@ -47,27 +16,9 @@
         <z><noise type="gaussian"><mean>0.0</mean><stddev>0.2</stddev></noise></z>
       </linear_acceleration>
-      <orientation>
-        <x><noise type="gaussian"><mean>0.0</mean><stddev>0.002</stddev></noise></x>
-        <y><noise type="gaussian"><mean>0.0</mean><stddev>0.002</stddev></noise></y>
-        <z><noise type="gaussian"><mean>0.0</mean><stddev>0.002</stddev></noise></z>
-      </orientation>
     </imu>
-    <!-- ✅ This must go here — under <sensor>, not inside <plugin> -->
     <covariance>
-      <orientation>
-        0.0025 0 0
-        0 0.0025 0
-        0 0 0.0025
-      </orientation>
-      <angular_velocity>
-        0.000225 0 0
-        0 0.000225 0
-        0 0 0.000225
-      </angular_velocity>
-      <linear_acceleration>
-        0.04 0 0
-        0 0.04 0
-        0 0 0.04
-      </linear_acceleration>
+      <orientation>0.0004 0 0 0 0.0004 0 0 0 0.0004</orientation>
+      <angular_velocity>0.0001 0 0 0 0.0001 0 0 0 0.0001</angular_velocity>
+      <linear_acceleration>0.05 0 0 0 0.05 0 0 0 0.05</linear_acceleration>
     </covariance>
     <plugin name="imu_plugin" filename="libgazebo_ros_imu_sensor.so">
@@ -80,3 +31,2 @@
   </sensor>
 </gazebo>
-</robot>

File: description/lidar.xacro (robot description, xacro)
@@ -1,52 +1,54 @@
 <?xml version="1.0"?>
-<robot xmlns:xacro="http://www.ros.org/wiki/xacro" >
+<robot xmlns:xacro="http://www.ros.org/wiki/xacro">
+  <xacro:macro name="lidar_sensor" params="parent">
     <joint name="laser_joint" type="fixed">
-        <parent link="chassis"/>
-        <child link="laser_frame"/>
-        <origin xyz="0.1 0 0.175" rpy="0 0 0"/>
+      <parent link="${parent}"/>
+      <child link="laser_frame"/>
+      <origin xyz="0.1 0 0.175" rpy="0 0 0"/>
     </joint>
     <link name="laser_frame">
-        <visual>
-            <geometry>
-                <cylinder radius="0.05" length="0.04"/>
-            </geometry>
-            <material name="red"/>
-        </visual>
-        <collision>
-            <geometry>
-                <cylinder radius="0.05" length="0.04"/>
-            </geometry>
-        </collision>
-        <xacro:inertial_cylinder mass="0.1" length="0.04" radius="0.05">
-            <origin xyz="0 0 0" rpy="0 0 0"/>
-        </xacro:inertial_cylinder>
+      <visual>
+        <geometry>
+          <cylinder radius="0.05" length="0.04"/>
+        </geometry>
+        <material name="red"/>
+      </visual>
+      <collision>
+        <geometry>
+          <cylinder radius="0.05" length="0.04"/>
+        </geometry>
+      </collision>
+      <xacro:inertial_cylinder mass="0.1" length="0.04" radius="0.05">
+        <origin xyz="0 0 0" rpy="0 0 0"/>
+      </xacro:inertial_cylinder>
     </link>
     <gazebo reference="laser_frame">
-        <material>Gazebo/Red</material>
-        <sensor name="laser" type="ray">
-            <pose> 0 0 0 0 0 0 </pose>
-            <visualize>true</visualize>
-            <update_rate>10</update_rate>
-            <ray>
-                <scan>
-                    <horizontal>
-                        <samples>360</samples>
-                        <min_angle>-3.14</min_angle>
-                        <max_angle>3.14</max_angle>
-                    </horizontal>
-                </scan>
-                <range>
-                    <min>0.3</min>
-                    <max>12</max>
-                </range>
-            </ray>
-            <plugin name="laser_controller" filename="libgazebo_ros_ray_sensor.so">
-                <ros>
-                    <argument>~/out:=scan</argument>
-                </ros>
-                <output_type>sensor_msgs/LaserScan</output_type>
-                <frame_name>laser_frame</frame_name>
-            </plugin>
-        </sensor>
+      <material>Gazebo/Red</material>
+      <sensor name="laser" type="ray">
+        <pose>0 0 0 0 0 0</pose>
+        <visualize>false</visualize>
+        <update_rate>10</update_rate>
+        <ray>
+          <scan>
+            <horizontal>
+              <samples>360</samples>
+              <min_angle>-3.14</min_angle>
+              <max_angle>3.14</max_angle>
+            </horizontal>
+          </scan>
+          <range>
+            <min>0.3</min>
+            <max>12.0</max>
+          </range>
+        </ray>
+        <plugin name="laser_controller" filename="libgazebo_ros_ray_sensor.so">
+          <ros>
+            <argument>~/out:=scan</argument>
+          </ros>
+          <output_type>sensor_msgs/LaserScan</output_type>
+          <frame_name>laser_frame</frame_name>
+        </plugin>
+      </sensor>
     </gazebo>
+  </xacro:macro>
 </robot>

File: description/robot.urdf.xacro (robot description, xacro)
@@ -1,4 +1,4 @@
 <?xml version="1.0"?>
-<robot xmlns:xacro="http://www.ros.org/wiki/xacro"  name="robot">
+<robot xmlns:xacro="http://www.ros.org/wiki/xacro" name="robot">
     <xacro:arg name="use_ros2_control" default="true"/>
     <xacro:include filename="robot_core.xacro" />
@@ -9,8 +9,8 @@
         <xacro:include filename="gazebo_control.xacro" />
     </xacro:unless>
+    <!-- 🔄 Include and call lidar macro here -->
     <xacro:include filename="lidar.xacro" />
+    <xacro:lidar_sensor parent="chassis"/>
     <xacro:include filename="camera.xacro" />
     <xacro:include filename="imu.xacro" />
-    <!-- <xacro:include filename="depth_camera.xacro" /> -->
-    <!--xacro:include filename="face.xacro" /> -->
 </robot>

File: description/robot_core.xacro (robot description, xacro)
@@ -32,6 +32,5 @@
     </material>
     <!-- BASE LINK -->
-    <link name="base_link">
-    </link>
+    <link name="base_link"/>
     <!-- BASE_FOOTPRINT LINK -->
     <joint name="base_footprint_joint" type="fixed">
@@ -40,6 +39,5 @@
         <origin xyz="0 0 0" rpy="0 0 0"/>
     </joint>
-    <link name="base_footprint">
-    </link>
+    <link name="base_footprint"/>
     <!-- CHASSIS LINK -->
     <joint name="chassis_joint" type="fixed">
@@ -67,5 +65,5 @@
     </link>
     <gazebo reference="chassis">
-        <material>Gazebo/Orange</material>
+        <material>Gazebo/white</material>
     </gazebo>
     <!-- LEFT WHEEL LINK -->
@@ -93,5 +91,5 @@
     </link>
     <gazebo reference="left_wheel">
-        <material>Gazebo/Blue</material>
+        <material>Gazebo/black</material>
     </gazebo>
     <!-- RIGHT WHEEL LINK -->
@@ -119,5 +117,5 @@
     </link>
     <gazebo reference="right_wheel">
-        <material>Gazebo/Blue</material>
+        <material>Gazebo/black</material>
     </gazebo>
     <!-- CASTER WHEEL LINK -->
@@ -144,5 +142,5 @@
     </link>
     <gazebo reference="caster_wheel">
-        <material>Gazebo/White</material>
+        <material>Gazebo/black</material>
         <mu1 value="0.001"/>
         <mu2 value="0.001"/>

Commit message: carto_and_toolbox

File: description/imu.xacro (robot description, xacro)
@@ -1,32 +1,61 @@
-<gazebo reference="imu_link">
-  <sensor name="imu_sensor" type="imu">
-    <always_on>true</always_on>
-    <update_rate>50</update_rate>
-    <visualize>true</visualize>
-    <imu>
-      <angular_velocity>
-        <z><noise type="gaussian"><mean>0.0</mean><stddev>0.01</stddev></noise></z>
-      </angular_velocity>
-      <orientation>
-        <z><noise type="gaussian"><mean>0.0</mean><stddev>0.001</stddev></noise></z>
-      </orientation>
-      <linear_acceleration>
-        <x><noise type="gaussian"><mean>0.0</mean><stddev>0.2</stddev></noise></x>
-        <y><noise type="gaussian"><mean>0.0</mean><stddev>0.2</stddev></noise></y>
-        <z><noise type="gaussian"><mean>0.0</mean><stddev>0.2</stddev></noise></z>
-      </linear_acceleration>
-    </imu>
-    <covariance>
-      <orientation>0.0004 0 0 0 0.0004 0 0 0 0.0004</orientation>
-      <angular_velocity>0.0001 0 0 0 0.0001 0 0 0 0.0001</angular_velocity>
-      <linear_acceleration>0.05 0 0 0 0.05 0 0 0 0.05</linear_acceleration>
-    </covariance>
-    <plugin name="imu_plugin" filename="libgazebo_ros_imu_sensor.so">
-      <ros>
-        <remapping>~/out:=/imu</remapping>
-      </ros>
+<?xml version="1.0"?>
+<robot xmlns:xacro="http://www.ros.org/wiki/xacro">
+  <!-- IMU Link -->
+  <link name="imu_link">
+    <visual>
+      <origin xyz="0 0 0" rpy="0 0 0"/>
+      <geometry><box size="0.03 0.03 0.01"/></geometry>
+      <material name="black"/>
+    </visual>
+    <collision>
+      <origin xyz="0 0 0" rpy="0 0 0"/>
+      <geometry><box size="0.03 0.03 0.01"/></geometry>
+    </collision>
+    <inertial>
+      <mass value="0.01"/>
+      <origin xyz="0 0 0" rpy="0 0 0"/>
+      <inertia ixx="1e-6" ixy="0" ixz="0" iyy="1e-6" iyz="0" izz="1e-6"/>
+    </inertial>
+  </link>
+  <!-- IMU Joint -->
+  <joint name="imu_joint" type="fixed">
+    <parent link="chassis"/>
+    <child link="imu_link"/>
+    <origin xyz="0.0 0.0 0.08" rpy="0 0 0"/>
+  </joint>
+  <!-- Gazebo IMU Sensor -->
+  <gazebo reference="imu_link">
+    <sensor name="imu_sensor" type="imu">
+      <always_on>true</always_on>
       <update_rate>50</update_rate>
-      <frame_name>imu_link</frame_name>
-    </plugin>
-  </sensor>
-</gazebo>
+      <visualize>true</visualize>
+      <imu>
+        <angular_velocity>
+          <x><noise type="gaussian"><mean>0.0</mean><stddev>0.01</stddev></noise></x>
+          <y><noise type="gaussian"><mean>0.0</mean><stddev>0.01</stddev></noise></y>
+          <z><noise type="gaussian"><mean>0.0</mean><stddev>0.01</stddev></noise></z>
+        </angular_velocity>
+        <orientation>
+          <x><noise type="gaussian"><mean>0.0</mean><stddev>0.001</stddev></noise></x>
+          <y><noise type="gaussian"><mean>0.0</mean><stddev>0.001</stddev></noise></y>
+          <z><noise type="gaussian"><mean>0.0</mean><stddev>0.001</stddev></noise></z>
+        </orientation>
+        <linear_acceleration>
+          <x><noise type="gaussian"><mean>0.0</mean><stddev>0.2</stddev></noise></x>
+          <y><noise type="gaussian"><mean>0.0</mean><stddev>0.2</stddev></noise></y>
+          <z><noise type="gaussian"><mean>0.0</mean><stddev>0.2</stddev></noise></z>
+        </linear_acceleration>
+      </imu>
+      <covariance>
+        <orientation>0.0004 0 0 0 0.0004 0 0 0 0.0004</orientation>
+        <angular_velocity>0.0001 0 0 0 0.0001 0 0 0 0.0001</angular_velocity>
+        <linear_acceleration>0.05 0 0 0 0.05 0 0 0 0.05</linear_acceleration>
+      </covariance>
+      <plugin name="imu_plugin" filename="libgazebo_ros_imu_sensor.so">
+        <ros><remapping>~/out:=/imu</remapping></ros>
+        <update_rate>50</update_rate>
+        <frame_name>imu_link</frame_name>
+      </plugin>
+    </sensor>
+  </gazebo>
+</robot>
